File: volatgeprobe.kicad_pcb (KiCad board)
At the start: 2 copper layers, 107 x 49 mm, 52 parts, among them IC1 AMC1301SDWV, J1 Conn_01x01_Male, J2 Conn_01x01_Male, J3 Conn_01x02_Male, J4 Conn_Coaxial, SW1 SW_SPST, U1 AZ1117IH-3.3TRG1, U4 LF353M, U5 LF353M

Commit message: shorted ldo outs
Parts:
- 111: renamed from 5V-5V Iso
- U2: renamed from 5V-15V Iso
- renumbered LED to D1
Connections:
- U1 pad 2: unconnected-(U1-OUTPUT-Pad2) -> +5V_re
Routing:
- net +5V_re: track 70.3 -> 76.5 mm
Changed lines of the file:
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@@
   (net 33 "Net-(SW1-B)")
   (net 34 "Net-(R20-Pad2)")
-  (net 35 "unconnected-(U1-OUTPUT-Pad2)")
-  (net 36 "Net-(U5-NEGB)")
+  (net 35 "Net-(U5-NEGB)")
   (footprint "22uf:EEE0GA101SR" (layer "F.Cu")
     (at 133.51625 111.11)
@@
       (net 2 "GND") (pinfunction "POSB") (pintype "input"))
     (pad "6" smd roundrect (at 2.47 0.635) (size 1.97 0.6) (layers "F.Cu" "F.Paste" "F.Mask") (roundrect_rratio 0.07)
-      (net 36 "Net-(U5-NEGB)") (pinfunction "NEGB") (pintype "input"))
+      (net 35 "Net-(U5-NEGB)") (pinfunction "NEGB") (pintype "input"))
     (pad "7" smd roundrect (at 2.47 -0.635) (size 1.97 0.6) (layers "F.Cu" "F.Paste" "F.Mask") (roundrect_rratio 0.07)
       (net 24 "Net-(J4-In)") (pinfunction "OUTB") (pintype "output"))
@@
     (property "ki_keywords" "LED diode")
     (attr through_hole)
-    (fp_text reference "LED" (at 1.41 -4.79) (layer "F.SilkS")
+    (fp_text reference "D1" (at 1.41 -4.79) (layer "F.SilkS")
         (effects (font (size 1 1) (thickness 0.15)))
     )
@@
     (property "Sheetname" "")
     (attr through_hole)
-    (fp_text reference "5V-15V Iso" (at -2.9325 7.5725) (layer "F.SilkS")
+    (fp_text reference "U2" (at -2.9325 7.5725) (layer "F.SilkS")
         (effects (font (size 1 1) (thickness 0.15)))
     )
@@
     (property "ki_description" "DC DC CONVERTER 5V 1W")
     (attr through_hole)
-    (fp_text reference "5V-5V Iso" (at 7.235 3.325) (layer "F.SilkS")
+    (fp_text reference "111" (at 7.235 3.325) (layer "F.SilkS")
         (effects (font (size 1.27 1.27) (thickness 0.254)))
     )
@@
       (net 6 "GND1") (pinfunction "GND") (pintype "power_in"))
     (pad "2" smd rect (at -3.1 0 180) (size 2.2 1.2) (layers "F.Cu" "F.Paste" "F.Mask")
-      (net 35 "unconnected-(U1-OUTPUT-Pad2)") (pinfunction "OUTPUT") (pintype "output+no_connect"))
+      (net 7 "+5V_re") (pinfunction "OUTPUT") (pintype "output"))
     (pad "3" smd rect (at -3.1 2.3 180) (size 2.2 1.2) (layers "F.Cu" "F.Paste" "F.Mask")
       (net 33 "Net-(SW1-B)") (pinfunction "INPUT") (pintype "input"))
@@
       (net 29 "Net-(R18-Pad1)") (pintype "bidirectional"))
     (pad "2" thru_hole circle (at 0 0) (size 1.508 1.508) (drill 1) (layers "*.Cu" "*.Mask")
-      (net 36 "Net-(U5-NEGB)") (pintype "bidirectional"))
+      (net 35 "Net-(U5-NEGB)") (pintype "bidirectional"))
     (pad "3" thru_hole circle (at 2.5 0) (size 1.508 1.508) (drill 1) (layers "*.Cu" "*.Mask")
       (net 30 "Net-(R19-Pad1)") (pintype "bidirectional"))
@@
   (segment (start 154.01625 108.65) (end 154.01625 112.095) (width 0.25) (layer "B.Cu") (net 5))
   (segment (start 132.90125 108.345) (end 135.66625 111.11) (width 0.25) (layer "F.Cu") (net 6))
+  (segment (start 135.66625 111.11) (end 138.21625 113.66) (width 0.25) (layer "F.Cu") (net 6))
   (segment (start 143.22375 112.7275) (end 143.22375 120.0675) (width 0.25) (layer "F.Cu") (net 6))
   (segment (start 126.58625 121.41) (end 136.36625 121.41) (width 0.25) (layer "F.Cu") (net 6))
@@
   (segment (start 132.90125 104.175) (end 132.90125 108.345) (width 0.25) (layer "F.Cu") (net 6))
   (segment (start 129.69625 83.59) (end 129.72625 83.56) (width 0.4) (layer "F.Cu") (net 6))
-  (segment (start 135.66625 111.11) (end 134.01625 112.76) (width 0.25) (layer "F.Cu") (net 6))
+  (segment (start 138.21625 113.66) (end 138.21625 120.08) (width 0.25) (layer "F.Cu") (net 6))
   (segment (start 136.29625 110.48) (end 141.41625 110.48) (width 0.25) (layer "F.Cu") (net 6))
   (segment (start 122.99625 125) (end 126.58625 121.41) (width 0.25) (layer "F.Cu") (net 6))
-  (segment (start 134.01625 112.76) (end 134.01625 120.38) (width 0.25) (layer "F.Cu") (net 6))
   (segment (start 132.90125 86.735) (end 132.90125 96.61) (width 0.25) (layer "F.Cu") (net 6))
   (segment (start 135.48625 109.21) (end 135.48625 110.93) (width 0.4) (layer "F.Cu") (net 6))
   (segment (start 132.90125 98.97) (end 132.90125 104.175) (width 0.25) (layer "F.Cu") (net 6))
+  (segment (start 136.88625 121.41) (end 136.36625 121.41) (width 0.25) (layer "F.Cu") (net 6))
   (segment (start 132.90125 104.175) (end 131.60125 105.475) (width 0.25) (layer "F.Cu") (net 6))
   (segment (start 135.48625 110.93) (end 135.66625 111.11) (width 0.4) (layer "F.Cu") (net 6))
@@
   (segment (start 141.41625 110.48) (end 143.22375 112.2875) (width 0.25) (layer "F.Cu") (net 6))
   (segment (start 129.72625 83.56) (end 132.90125 86.735) (width 0.25) (layer "F.Cu") (net 6))
-  (segment (start 134.01625 120.38) (end 135.04625 121.41) (width 0.25) (layer "F.Cu") (net 6))
+  (segment (start 138.21625 120.08) (end 136.88625 121.41) (width 0.25) (layer "F.Cu") (net 6))
   (segment (start 121.41625 125) (end 122.99625 125) (width 0.25) (layer "F.Cu") (net 6))
   (segment (start 132.90125 96.61) (end 132.90125 98.97) (width 0.25) (layer "F.Cu") (net 6))
   (segment (start 131.60125 105.475) (end 131.00125 105.475) (width 0.25) (layer "F.Cu") (net 6))
-  (segment (start 135.04625 121.41) (end 136.36625 121.41) (width 0.25) (layer "F.Cu") (net 6))
   (via (at 135.48625 109.21) (size 0.8) (drill 0.4) (layers "F.Cu" "B.Cu") (net 6))
   (via (at 127.91625 83.59) (size 0.8) (drill 0.4) (layers "F.Cu" "B.Cu") (net 6))
@@
   (segment (start 129.30625 110.97) (end 131.22625 110.97) (width 0.25) (layer "F.Cu") (net 7))
   (segment (start 140.68375 120.0675) (end 141.40125 120.785) (width 0.25) (layer "F.Cu") (net 7))
+  (segment (start 130.16625 119.11) (end 136.36625 119.11) (width 0.25) (layer "F.Cu") (net 7))
   (segment (start 124.97625 119.11) (end 130.16625 119.11) (width 0.25) (layer "F.Cu") (net 7))
   (segment (start 131.36625 112.25) (end 131.36625 111.11) (width 0.25) (layer "F.Cu") (net 7))
@@
   (segment (start 160.51625 100.4475) (end 159.01625 101.9475) (width 0.25) (layer "F.Cu") (net 34))
   (segment (start 160.51625 99.01475) (end 160.51625 100.4475) (width 0.25) (layer "F.Cu") (net 34))
-  (segment (start 168.33625 108.15) (end 168.24125 108.245) (width 0.3) (layer "F.Cu") (net 36))
-  (segment (start 168.24125 108.245) (end 166.73625 108.245) (width 0.3) (layer "F.Cu") (net 36))
-  (via (at 168.33625 108.15) (size 0.8) (drill 0.4) (layers "F.Cu" "B.Cu") (net 36))
-  (segment (start 168.33625 108.15) (end 169.31625 108.15) (width 0.3) (layer "B.Cu") (net 36))
-  (segment (start 169.31625 108.15) (end 177.50625 99.96) (width 0.3) (layer "B.Cu") (net 36))
-  (segment (start 177.50625 99.96) (end 177.50625 99.1) (width 0.3) (layer "B.Cu") (net 36))
+  (segment (start 168.33625 108.15) (end 168.24125 108.245) (width 0.3) (layer "F.Cu") (net 35))
+  (segment (start 168.24125 108.245) (end 166.73625 108.245) (width 0.3) (layer "F.Cu") (net 35))
+  (via (at 168.33625 108.15) (size 0.8) (drill 0.4) (layers "F.Cu" "B.Cu") (net 35))
+  (segment (start 168.33625 108.15) (end 169.31625 108.15) (width 0.3) (layer "B.Cu") (net 35))
+  (segment (start 169.31625 108.15) (end 177.50625 99.96) (width 0.3) (layer "B.Cu") (net 35))
+  (segment (start 177.50625 99.96) (end 177.50625 99.1) (width 0.3) (layer "B.Cu") (net 35))
   (zone (net 2) (net_name "GND") (layer "F.Cu") (hatch edge 0.5)
     (connect_pads (clearance 0.508))

Commit message: changed
Other:
- board size 107 x 49 mm -> 106.9 x 49.2 mm
Changed lines of the file:
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@@
     (property "ki_keywords" "connector")
     (attr through_hole)
-    (fp_text reference "J2" (at 0.72 3.105 180) (layer "F.SilkS")
+    (fp_text reference "J2" (at -0.61 4.045 180) (layer "F.SilkS")
         (effects (font (size 1.27 1.27) (thickness 0.254)))
     )
@@
     (property "ki_keywords" "connector")
     (attr through_hole)
-    (fp_text reference "J1" (at 0.9025 3.35) (layer "F.SilkS")
+    (fp_text reference "J1" (at -0.5875 -4.36) (layer "F.SilkS")
         (effects (font (size 1.27 1.27) (thickness 0.254)))
     )
@@
       (solder_mask_margin 0.1016))
   )
-  (gr_arc (start 96.76625 84.71) (mid 98.184413 81.598526) (end 101.267142 80.118919)
+  (gr_arc (start 101.93625 129.1) (mid 98.400716 127.635534) (end 96.93625 124.1)
     (stroke (width 0.1) (type default)) (layer "Edge.Cuts"))
-  (gr_line (start 101.267142 80.118919) (end 198.51625 80.25608)
+  (gr_arc (start 96.93625 84.94) (mid 98.400719 81.404484) (end 101.93625 79.94)
     (stroke (width 0.1) (type default)) (layer "Edge.Cuts"))
-  (gr_rect (start 98.05625 101.77) (end 122.75625 104.77)
+  (gr_line (start 198.83625 129.1) (end 101.93625 129.1)
+    (stroke (width 0.1) (type default)) (layer "Edge.Cuts"))
+  (gr_line (start 101.93625 79.94) (end 198.83625 79.94)
+    (stroke (width 0.1) (type default)) (layer "Edge.Cuts"))
+  (gr_arc (start 203.83625 124.1) (mid 202.371784 127.635534) (end 198.83625 129.1)
+    (stroke (width 0.1) (type default)) (layer "Edge.Cuts"))
+  (gr_rect (start 100.53625 101.77) (end 122.75625 104.77)
     (stroke (width 0.1) (type default)) (fill none) (layer "Edge.Cuts"))
-  (gr_arc (start 198.51625 80.25608) (mid 202.195298 81.822401) (end 203.61625 85.56)
+  (gr_arc (start 198.83625 79.94) (mid 202.371784 81.404466) (end 203.83625 84.94)
     (stroke (width 0.1) (type default)) (layer "Edge.Cuts"))
-  (gr_line (start 97.065682 123.86) (end 96.76625 84.71)
+  (gr_line (start 203.83625 84.94) (end 203.83625 124.1)
     (stroke (width 0.1) (type default)) (layer "Edge.Cuts"))
-  (gr_arc (start 101.94125 128.81) (mid 98.489253 127.333963) (end 97.065682 123.86)
-    (stroke (width 0.1) (type default)) (layer "Edge.Cuts"))
-  (gr_line (start 198.76625 129.11) (end 101.94125 128.81)
-    (stroke (width 0.1) (type default)) (layer "Edge.Cuts"))
-  (gr_arc (start 203.76625 124.11) (mid 202.301784 127.645534) (end 198.76625 129.11)
-    (stroke (width 0.1) (type default)) (layer "Edge.Cuts"))
-  (gr_line (start 203.61625 85.56) (end 203.76625 124.11)
+  (gr_line (start 96.93625 124.1) (end 96.93625 84.94)
     (stroke (width 0.1) (type default)) (layer "Edge.Cuts"))
   (gr_text "check banana jack size" (at 154.94625 70.07) (layer "Cmts.User")
