File: volatgeprobe.kicad_pcb (KiCad board)
At the start: 2 copper layers, 106.9 x 49.2 mm, 53 parts, among them IC1 AMC1301SDWV, J1 Conn_01x01_Male, J2 Conn_01x01_Male, J3 Conn_01x02_Male, J4 Conn_Coaxial, SW1 SW_SPST, U1 AZ1117IH-3.3TRG1, U2 5-15v, U4 LF353M, U5 LF353M

Commit message: battery_3D_added
Other:
- board text removed: "check banana jack size"
Changed lines of the file:
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@@
     (pad "3" thru_hole circle (at 36.3 9.65) (size 2.4 2.4) (drill 1.6) (layers "*.Cu" "*.Mask")
       (solder_mask_margin 0.1016))
+    (model "${KIPRJMOD}/Footprints&symbols/battery/BATTERY_holder.stp"
+      (offset (xyz 0 0 0))
+      (scale (xyz 1 1 1))
+      (rotate (xyz 0 0 0))
+    )
   )
   (gr_arc (start 101.93625 129.1) (mid 98.400716 127.635534) (end 96.93625 124.1)
@@
     (effects (font (size 1 1.5) (thickness 0.25) bold) (justify left bottom))
   )
-  (gr_text "check banana jack size" (at 154.94625 70.07) (layer "Cmts.User")
-    (effects (font (size 2 2) (thickness 0.25) bold) (justify left bottom))
-  )
   (segment (start 120.01625 89.4294) (end 127.04565 89.4294) (width 0.25) (layer "F.Cu") (net 1))
